File: _autosave-RPI.kicad_sch (KiCad schematic)
At the start: 24 parts, among them J1 Conn_01x02_Male, J1 GPIO, J2 Conn_02x12, J4 Conn_01x03, Q1 IRF9540N, U1 LM1085-5.0, U2 CAT24C256

Commit message: Added diode protection and switches
Connections:
- net +5V: no longer D?.2 (A), J1.2 (Pin_2)
- net +BATT: now also J?.1 (Pin_1)
- net VCC: no longer J?.1 (Pin_1)
- new net VD: D?.2 (A), J1.2 (Pin_2)
Changed lines of the file:
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@@
   (junction (at 259.08 143.51) (diameter 1.016) (color 0 0 0 0)
-  )
-  (junction (at 54.61 26.67) (diameter 1.016) (color 0 0 0 0)
   )
   (junction (at 246.38 156.21) (diameter 1.016) (color 0 0 0 0)
@@
     (stroke (width 0) (type default) (color 0 0 0 0))
   )
-  (wire (pts (xy 74.93 143.51) (xy 74.93 146.05))
-    (stroke (width 0) (type default) (color 0 0 0 0))
-  )
   (wire (pts (xy 90.17 85.09) (xy 88.9 85.09))
     (stroke (width 0) (type default) (color 0 0 0 0))
@@
     (stroke (width 0) (type solid) (color 0 0 0 0))
   )
+  (wire (pts (xy 72.39 146.05) (xy 74.93 146.05))
+    (stroke (width 0) (type default) (color 0 0 0 0))
+  )
   (wire (pts (xy 100.33 46.99) (xy 105.41 46.99))
     (stroke (width 0) (type solid) (color 0 0 0 0))
@@
     (stroke (width 0) (type default) (color 0 0 0 0))
   )
+  (wire (pts (xy 54.61 24.13) (xy 54.61 26.67))
+    (stroke (width 0) (type default) (color 0 0 0 0))
+  )
   (wire (pts (xy 102.87 36.83) (xy 102.87 44.45))
     (stroke (width 0) (type solid) (color 0 0 0 0))
@@
     (stroke (width 0) (type solid) (color 0 0 0 0))
   )
+  (wire (pts (xy 52.07 29.21) (xy 58.42 29.21))
+    (stroke (width 0) (type default) (color 0 0 0 0))
+  )
   (polyline (pts (xy 138.43 12.0144) (xy 138.43 68.58))
     (stroke (width 0) (type default) (color 0 0 0 0))
@@
     (stroke (width 0) (type default) (color 0 0 0 0))
   )
-  (wire (pts (xy 72.39 146.05) (xy 74.93 146.05))
-    (stroke (width 0) (type default) (color 0 0 0 0))
-  )
   (wire (pts (xy 148.59 82.55) (xy 132.08 82.55))
     (stroke (width 0) (type default) (color 0 0 0 0))
@@
     (stroke (width 0) (type solid) (color 0 0 0 0))
   )
+  (wire (pts (xy 74.93 146.05) (xy 74.93 144.78))
+    (stroke (width 0) (type default) (color 0 0 0 0))
+  )
   (wire (pts (xy 48.26 104.14) (xy 48.26 114.3))
     (stroke (width 0) (type default) (color 0 0 0 0))
@@
     (stroke (width 0) (type solid) (color 0 0 0 0))
   )
-  (wire (pts (xy 54.61 26.67) (xy 54.61 29.21))
-    (stroke (width 0) (type solid) (color 0 0 0 0))
-  )
   (polyline (pts (xy 80.01 119.38) (xy 80.01 172.72))
     (stroke (width 0) (type default) (color 0 0 0 0))
@@
     (stroke (width 0) (type default) (color 0 0 0 0))
   )
-  (wire (pts (xy 54.61 22.86) (xy 54.61 26.67))
-    (stroke (width 0) (type solid) (color 0 0 0 0))
-  )
   (wire (pts (xy 161.29 27.94) (xy 156.21 27.94))
     (stroke (width 0) (type default) (color 0 0 0 0))
@@
     (stroke (width 0) (type default) (color 0 0 0 0))
   )
-  (wire (pts (xy 54.61 29.21) (xy 52.07 29.21))
-    (stroke (width 0) (type solid) (color 0 0 0 0))
-  )
   (wire (pts (xy 48.26 127) (xy 45.72 127))
     (stroke (width 0) (type default) (color 0 0 0 0))
@@
   )
   (wire (pts (xy 90.17 87.63) (xy 88.9 87.63))
+    (stroke (width 0) (type default) (color 0 0 0 0))
+  )
+  (wire (pts (xy 58.42 24.13) (xy 58.42 29.21))
     (stroke (width 0) (type default) (color 0 0 0 0))
   )
@@
     (effects (font (size 1.27 1.27)) (justify right bottom))
   )
-  (symbol (lib_id "power:+5V") (at 54.61 22.86 0) (unit 1)
-    (in_bom yes) (on_board yes)
-    (property "Reference" "#PWR01" (id 0) (at 54.61 26.67 0)
-      (effects (font (size 1.27 1.27)) hide)
-    )
-    (property "Value" "+5V" (id 1) (at 54.9783 18.5356 0))
-    (property "Footprint" "" (id 2) (at 54.61 22.86 0))
-    (property "Datasheet" "" (id 3) (at 54.61 22.86 0))
+  (symbol (lib_id "power:+5V") (at 58.42 24.13 0) (unit 1)
+    (in_bom yes) (on_board yes)
+    (property "Reference" "#PWR01" (id 0) (at 58.42 27.94 0)
+      (effects (font (size 1.27 1.27)) hide)
+    )
+    (property "Value" "+5V" (id 1) (at 58.7883 19.8056 0))
+    (property "Footprint" "" (id 2) (at 58.42 24.13 0))
+    (property "Datasheet" "" (id 3) (at 58.42 24.13 0))
     (pin "1")
   )
@@
     (pin "2")
   )
+  (symbol (lib_id "power:VD") (at 54.61 24.13 0) (unit 1)
+    (in_bom yes) (on_board yes) (fields_autoplaced)
+    (property "Reference" "#PWR?" (id 0) (at 54.61 27.94 0)
+      (effects (font (size 1.27 1.27)) hide)
+    )
+    (property "Value" "VD" (id 1) (at 54.61 19.05 0))
+    (property "Footprint" "" (id 2) (at 54.61 24.13 0)
+      (effects (font (size 1.27 1.27)) hide)
+    )
+    (property "Datasheet" "" (id 3) (at 54.61 24.13 0)
+      (effects (font (size 1.27 1.27)) hide)
+    )
+    (pin "1")
+  )
   (symbol (lib_name "GND_1") (lib_id "power:GND") (at 31.75 115.57 0) (unit 1)
     (in_bom yes) (on_board yes) (fields_autoplaced)
@@
     )
     (property "Datasheet" "" (id 3) (at 31.75 115.57 0)
+      (effects (font (size 1.27 1.27)) hide)
+    )
+    (pin "1")
+  )
+  (symbol (lib_id "power:VD") (at 74.93 144.78 0) (unit 1)
+    (in_bom yes) (on_board yes) (fields_autoplaced)
+    (property "Reference" "#PWR?" (id 0) (at 74.93 148.59 0)
+      (effects (font (size 1.27 1.27)) hide)
+    )
+    (property "Value" "VD" (id 1) (at 74.93 139.7 0))
+    (property "Footprint" "" (id 2) (at 74.93 144.78 0)
+      (effects (font (size 1.27 1.27)) hide)
+    )
+    (property "Datasheet" "" (id 3) (at 74.93 144.78 0)
       (effects (font (size 1.27 1.27)) hide)
     )
@@
     (pin "2")
   )
-  (symbol (lib_id "power:+5V") (at 74.93 143.51 0) (unit 1)
-    (in_bom yes) (on_board yes)
-    (property "Reference" "#PWR?" (id 0) (at 74.93 147.32 0)
-      (effects (font (size 1.27 1.27)) hide)
-    )
-    (property "Value" "+5V" (id 1) (at 75.2983 139.1856 0))
-    (property "Footprint" "" (id 2) (at 74.93 143.51 0))
-    (property "Datasheet" "" (id 3) (at 74.93 143.51 0))
-    (pin "1")
-  )
   (symbol (lib_id "Device:C_Polarized_US") (at 60.96 157.48 0) (unit 1)
     (in_bom yes) (on_board yes) (fields_autoplaced)
@@
     (property "Footprint" "" (id 2) (at 120.65 57.15 0))
     (property "Datasheet" "" (id 3) (at 120.65 57.15 0))
-    (pin "1")
-  )
-  (symbol (lib_id "power:VCC") (at 88.9 85.09 0) (unit 1)
-    (in_bom yes) (on_board yes) (fields_autoplaced)
-    (property "Reference" "#PWR?" (id 0) (at 88.9 88.9 0)
-      (effects (font (size 1.27 1.27)) hide)
-    )
-    (property "Value" "VCC" (id 1) (at 88.9 80.01 0))
-    (property "Footprint" "" (id 2) (at 88.9 85.09 0)
-      (effects (font (size 1.27 1.27)) hide)
-    )
-    (property "Datasheet" "" (id 3) (at 88.9 85.09 0)
-      (effects (font (size 1.27 1.27)) hide)
-    )
     (pin "1")
   )
@@
     (pin "1")
   )
+  (symbol (lib_id "power:+BATT") (at 88.9 85.09 0) (unit 1)
+    (in_bom yes) (on_board yes) (fields_autoplaced)
+    (property "Reference" "#PWR?" (id 0) (at 88.9 88.9 0)
+      (effects (font (size 1.27 1.27)) hide)
+    )
+    (property "Value" "+BATT" (id 1) (at 88.9 80.01 0))
+    (property "Footprint" "" (id 2) (at 88.9 85.09 0)
+      (effects (font (size 1.27 1.27)) hide)
+    )
+    (property "Datasheet" "" (id 3) (at 88.9 85.09 0)
+      (effects (font (size 1.27 1.27)) hide)
+    )
+    (pin "1")
+  )
   (symbol (lib_id "Device:C_Polarized_US") (at 29.21 157.48 0) (unit 1)
     (in_bom yes) (on_board yes) (fields_autoplaced)
@@
       (reference "#PWR?") (unit 1) (value "GND") (footprint "")
     )
+    (path "/38dcc1db-3bcc-4a73-9089-a11109b9e201"
+      (reference "#PWR?") (unit 1) (value "VD") (footprint "")
+    )
     (path "/3fafb5e6-3e49-4d59-9f28-529ce9266826"
       (reference "#PWR?") (unit 1) (value "GND") (footprint "")
     )
+    (path "/41a03794-bcc2-4b48-a636-83b334c4c7e5"
+      (reference "#PWR?") (unit 1) (value "VD") (footprint "")
+    )
     (path "/46573456-51b1-4798-ad1b-19ff0599ede3"
       (reference "#PWR?") (unit 1) (value "GND") (footprint "")
@@
       (reference "#PWR?") (unit 1) (value "GND") (footprint "")
     )
-    (path "/7d96ce1b-d2fd-4db9-8388-5bf7c5156989"
-      (reference "#PWR?") (unit 1) (value "+5V") (footprint "")
-    )
     (path "/86f917b1-0912-46a4-b9af-5b4658a27ffc"
       (reference "#PWR?") (unit 1) (value "GND") (footprint "")
@@
       (reference "#PWR?") (unit 1) (value "GND") (footprint "")
     )
-    (path "/8c56a6b1-5cd7-4e0d-b5e5-c40704d869b1"
-      (reference "#PWR?") (unit 1) (value "VCC") (footprint "")
-    )
     (path "/8d86f8f7-ecbc-4cd3-8849-6ca13540335e"
       (reference "#PWR?") (unit 1) (value "+3.3V") (footprint "")
@@
       (reference "#PWR?") (unit 1) (value "GND") (footprint "")
     )
+    (path "/e8b902b1-0f0c-4140-aea0-0b3b4f3ad743"
+      (reference "#PWR?") (unit 1) (value "+BATT") (footprint "")
+    )
     (path "/f118ba3b-99e3-4e45-85ab-7912d5798d53"
