File: RPI.kicad_sch (KiCad schematic)
At the start: 29 parts, among them J1 Conn_01x02_Male, J2 GPIO, J5 Conn_01x06, J6 Conn_01x04, J7 Conn_01x03, J8 Conn_01x02, J9 Conn_01x02, Q1 IRF9540N, Q2 IRF9540N, Q3 BC856BDW1, SW1 SW_SPDT, SW2 SW_SPDT, U1 LM1085-ADJ, U2 LM1085-ADJ

Commit message: Added DMMT library
Parts:
- added Q4: DMMT5401-7-F, SOT95P285X140-6N, symbol DMMT5401-7-F:DMMT5401-7-F
Connections:
- no-connect marks 3 -> 9
Changed lines of the file:
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@@
   (junction (at 107.95 40.64) (diameter 0) (color 0 0 0 0)
   )
+  (no_connect (at 93.98 168.91))
   (no_connect (at 85.09 97.79))
+  (no_connect (at 120.65 163.83))
+  (no_connect (at 99.06 163.83))
   (no_connect (at 137.16 36.83))
+  (no_connect (at 99.06 173.99))
+  (no_connect (at 115.57 168.91))
   (no_connect (at 137.16 49.53))
+  (no_connect (at 120.65 173.99))
   (wire (pts (xy 36.83 57.15) (xy 36.83 74.93))
     (stroke (width 0) (type solid) (color 0 0 0 0))
@@
   (symbol (lib_id "power:VCC") (at 99.06 123.19 0) (unit 1)
     (in_bom yes) (on_board yes) (fields_autoplaced)
-    (property "Reference" "#PWR?" (id 0) (at 99.06 127 0)
+    (property "Reference" "#PWR0127" (id 0) (at 99.06 127 0)
       (effects (font (size 1.27 1.27)) hide)
     )
@@
     (pin "1")
     (pin "2")
+  )
+  (symbol (lib_id "DMMT5401-7-F:DMMT5401-7-F") (at 118.11 168.91 0) (unit 2)
+    (in_bom yes) (on_board yes) (fields_autoplaced)
+    (property "Reference" "Q4" (id 0) (at 121.92 167.6129 0)
+      (effects (font (size 1.27 1.27)) (justify left))
+    )
+    (property "Value" "DMMT5401-7-F" (id 1) (at 121.92 170.1529 0)
+      (effects (font (size 1.27 1.27)) (justify left))
+    )
+    (property "Footprint" "SOT95P285X140-6N" (id 2) (at 118.11 168.91 0)
+      (effects (font (size 1.27 1.27)) (justify bottom) hide)
+    )
+    (property "Datasheet" "" (id 3) (at 118.11 168.91 0)
+      (effects (font (size 1.27 1.27)) hide)
+    )
+    (property "MANUFACTURER" "Diodes Inc." (id 4) (at 118.11 168.91 0)
+      (effects (font (size 1.27 1.27)) (justify bottom) hide)
+    )
+    (property "PARTREV" "8" (id 5) (at 118.11 168.91 0)
+      (effects (font (size 1.27 1.27)) (justify bottom) hide)
+    )
+    (property "STANDARD" "IPC7351B" (id 6) (at 118.11 168.91 0)
+      (effects (font (size 1.27 1.27)) (justify bottom) hide)
+    )
+    (pin "1")
+    (pin "2")
+    (pin "6")
+    (pin "3")
+    (pin "4")
+    (pin "5")
   )
   (symbol (lib_id "Connector_Generic:Conn_01x06") (at 58.42 105.41 180) (unit 1)
@@
     (pin "1")
   )
+  (symbol (lib_id "DMMT5401-7-F:DMMT5401-7-F") (at 96.52 168.91 0) (unit 1)
+    (in_bom yes) (on_board yes) (fields_autoplaced)
+    (property "Reference" "Q4" (id 0) (at 100.33 167.6129 0)
+      (effects (font (size 1.27 1.27)) (justify left))
+    )
+    (property "Value" "DMMT5401-7-F" (id 1) (at 100.33 170.1529 0)
+      (effects (font (size 1.27 1.27)) (justify left))
+    )
+    (property "Footprint" "SOT95P285X140-6N" (id 2) (at 96.52 168.91 0)
+      (effects (font (size 1.27 1.27)) (justify bottom) hide)
+    )
+    (property "Datasheet" "" (id 3) (at 96.52 168.91 0)
+      (effects (font (size 1.27 1.27)) hide)
+    )
+    (property "MANUFACTURER" "Diodes Inc." (id 4) (at 96.52 168.91 0)
+      (effects (font (size 1.27 1.27)) (justify bottom) hide)
+    )
+    (property "PARTREV" "8" (id 5) (at 96.52 168.91 0)
+      (effects (font (size 1.27 1.27)) (justify bottom) hide)
+    )
+    (property "STANDARD" "IPC7351B" (id 6) (at 96.52 168.91 0)
+      (effects (font (size 1.27 1.27)) (justify bottom) hide)
+    )
+    (pin "1")
+    (pin "2")
+    (pin "6")
+    (pin "3")
+    (pin "4")
+    (pin "5")
+  )
   (symbol (lib_name "GND_1") (lib_id "power:GND") (at 52.07 132.08 0) (unit 1)
     (in_bom yes) (on_board yes) (fields_autoplaced)
@@
   (symbol (lib_name "GND_1") (lib_id "power:GND") (at 135.89 140.97 0) (unit 1)
     (in_bom yes) (on_board yes) (fields_autoplaced)
-    (property "Reference" "#PWR?" (id 0) (at 135.89 147.32 0)
+    (property "Reference" "#PWR0117" (id 0) (at 135.89 147.32 0)
       (effects (font (size 1.27 1.27)) hide)
     )
@@
   (symbol (lib_name "GND_1") (lib_id "power:GND") (at 127 140.97 0) (unit 1)
     (in_bom yes) (on_board yes) (fields_autoplaced)
-    (property "Reference" "#PWR?" (id 0) (at 127 147.32 0)
+    (property "Reference" "#PWR0120" (id 0) (at 127 147.32 0)
       (effects (font (size 1.27 1.27)) hide)
     )
@@
   (symbol (lib_name "GND_1") (lib_id "power:GND") (at 102.87 140.97 0) (unit 1)
     (in_bom yes) (on_board yes) (fields_autoplaced)
-    (property "Reference" "#PWR?" (id 0) (at 102.87 147.32 0)
+    (property "Reference" "#PWR0126" (id 0) (at 102.87 147.32 0)
       (effects (font (size 1.27 1.27)) hide)
     )
@@
   (symbol (lib_id "power:Vdrive") (at 142.7082 123.19 0) (unit 1)
     (in_bom yes) (on_board yes) (fields_autoplaced)
-    (property "Reference" "#PWR?" (id 0) (at 137.6282 127 0)
+    (property "Reference" "#PWR0102" (id 0) (at 137.6282 127 0)
       (effects (font (size 1.27 1.27)) hide)
     )
@@
       (reference "#PWR0101") (unit 1) (value "GND") (footprint "")
     )
+    (path "/a94f3d14-8064-4aeb-8007-47d60c4f6721"
+      (reference "#PWR0102") (unit 1) (value "Vdrive") (footprint "")
+    )
     (path "/e0dc823d-0c24-4046-9bc5-77dfb982fea5"
       (reference "#PWR0103") (unit 1) (value "VCC") (footprint "")
@@
       (reference "#PWR0116") (unit 1) (value "+BATT") (footprint "")
     )
+    (path "/6c5c92cf-ed04-455a-a8a6-ddb87441b3fc"
+      (reference "#PWR0117") (unit 1) (value "GND") (footprint "")
+    )
     (path "/5e32a9e3-4050-4e82-9158-04afccf7328e"
       (reference "#PWR0118") (unit 1) (value "GND") (footprint "")
@@
       (reference "#PWR0119") (unit 1) (value "GND") (footprint "")
     )
+    (path "/710640b1-3629-4d16-acc9-e0df4be2282f"
+      (reference "#PWR0120") (unit 1) (value "GND") (footprint "")
+    )
     (path "/359b38cb-4c7c-485c-966f-750aa5e46f10"
       (reference "#PWR0121") (unit 1) (value "VD") (footprint "")
@@
       (reference "#PWR0125") (unit 1) (value "VDDF") (footprint "")
     )
+    (path "/8cb6bccf-20f5-44a2-83c4-6d17db5ca960"
+      (reference "#PWR0126") (unit 1) (value "GND") (footprint "")
+    )
+    (path "/05f42738-c4f2-4ba7-aea5-0abcd877790b"
+      (reference "#PWR0127") (unit 1) (value "VCC") (footprint "")
+    )
     (path "/cdb3726e-c1bd-48e1-b03b-f9a827b4631d"
       (reference "#PWR0135") (unit 1) (value "GND") (footprint "")
@@
       (reference "#PWR0137") (unit 1) (value "GND") (footprint "")
     )
-    (path "/05f42738-c4f2-4ba7-aea5-0abcd877790b"
-      (reference "#PWR?") (unit 1) (value "VCC") (footprint "")
-    )
-    (path "/6c5c92cf-ed04-455a-a8a6-ddb87441b3fc"
-      (reference "#PWR?") (unit 1) (value "GND") (footprint "")
-    )
-    (path "/710640b1-3629-4d16-acc9-e0df4be2282f"
-      (reference "#PWR?") (unit 1) (value "GND") (footprint "")
-    )
-    (path "/8cb6bccf-20f5-44a2-83c4-6d17db5ca960"
-      (reference "#PWR?") (unit 1) (value "GND") (footprint "")
-    )
-    (path "/a94f3d14-8064-4aeb-8007-47d60c4f6721"
-      (reference "#PWR?") (unit 1) (value "Vdrive") (footprint "")
-    )
     (path "/f0184481-2811-4caf-b158-2161fd534a7f"
       (reference "C1") (unit 1) (value "10u") (footprint "Capacitor_THT:CP_Radial_D5.0mm_P2.50mm")
@@
       (reference "Q3") (unit 2) (value "BC856BDW1") (footprint "Package_TO_SOT_SMD:SOT-363_SC-70-6")
     )
+    (path "/448c1e76-05c4-4345-93d8-55bc24339199"
+      (reference "Q4") (unit 1) (value "DMMT5401-7-F") (footprint "SOT95P285X140-6N")
+    )
+    (path "/0e622e6b-6509-43b3-a9d2-994fed504ebe"
+      (reference "Q4") (unit 2) (value "DMMT5401-7-F") (footprint "SOT95P285X140-6N")
+    )
     (path "/38ef363a-7814-447e-8937-52cf03fa7bcc"

Commit message: V2 Ready for checking
Parts:
- removed Q3: BC856BDW1, Package_TO_SOT_SMD:SOT-363_SC-70-6, symbol Transistor_BJT:BC856BDW1
- U1, U2: footprint RPi_Hat:LM1085-5.0 -> Package_TO_SOT_THT:TO-220-3_Vertical
Connections:
- net VD: now also Q4.5
- net VDDA: now also Q4.6
- net at Q4.3: now also Q4.1, Q4.2, R5.1
- net at Q4.4: now also Q2.1 (G), R6.1
- no-connect marks 9 -> 3
Other:
- moved on the sheet: Q4A, Q4B
